File: tests/visual_output/test_circuit.kicad_sch (KiCad schematic)
At the start: 2 parts

Commit message: feat: implement comprehensive KiCad component layout and pin-level connectivity system (#8)
* feat: implement comprehensive KiCad component layout and pin-level connectivity system

This commit implements a complete solution for KiCad schematic component positioning and wire connectivity issues (addresses Issues #2, #3, #4):

## Core Implementation

### Updated KiCad File Format Version (Issue #2)
- Updated all schematic files from outdated 20230121 to current 20240618 format
- Ensured compatibility with KiCad 8.0 and later versions
- Updated across all modules: sexpr_generator, circuit_tools, examples, and test fixtures

### ComponentLayoutManager System (Issue #3)
- Implemented comprehensive component boundary validation
- Added automatic positioning for components outside schematic boundaries
- Features: grid snapping, collision detection, multiple layout strategies
- Supports A4 schematic bounds with configurable margins and spacing

### ComponentPinMapper System (Issue #4)
- Implemented pin-level connectivity tracking and validation
- Added wire routing algorithms with orthogonal routing strategies
- Features: pin compatibility checking, connection point calculation, bus routing
- Supports standard component pin layouts (resistors, LEDs, power symbols, etc.)

### S-Expression Generator Integration
- Integrated both layout manager and pin mapper into schematic generation
- Added position validation and correction during schematic creation
- Implemented pin-level wire routing with proper connection points
- Added support for advanced multi-pin net routing

## Testing Infrastructure

### Test-Driven Development Documentation
- Added comprehensive TDD guidelines to CLAUDE.md and README.md
- Documented mandatory TDD workflow: RED → GREEN → REFACTOR
- Provided clear test commands and structure documentation

### Comprehensive Test Suite
- Created 32 unit tests for ComponentLayoutManager functionality
- Created 12 unit tests for ComponentPinMapper functionality
- Crea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
Parts:
- LED1: value Red LED -> Red
- R1: value 330Ω -> 1kΩ
Other:
- title: LED Blinker Test -> Visualization Test Circuit
Changed lines of the file:
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@@
   (paper "A4")
   (title_block
-    (title "LED Blinker Test")
+    (title "Visualization Test Circuit")
     (date "")
     (rev "")
     (company "")
   )
-  (symbol (lib_id "Device:R") (at 508.0 508.0 0) (unit 1)
+  (symbol (lib_id "Device:R") (at 500 500 0) (unit 1)
     (exclude_from_sim no) (in_bom yes) (on_board yes) (dnp no)
-    (property "Reference" "R1" (at 533.4 495.3 0))
-    (property "Value" "330Ω" (at 533.4 520.7 0))
-    (property "Footprint" "" (at 508.0 508.0 0))
-    (property "Datasheet" "~" (at 508.0 508.0 0))
+    (property "Reference" "R1" (at 525.4 487.3 0))
+    (property "Value" "1kΩ" (at 525.4 512.7 0))
+    (property "Footprint" "" (at 500 500 0))
+    (property "Datasheet" "~" (at 500 500 0))
     (pin "1")
     (pin "2")
   )
-  (symbol (lib_id "Device:LED") (at 1016.0 508.0 0) (unit 1)
+  (symbol (lib_id "Device:LED") (at 1000 500 0) (unit 1)
     (exclude_from_sim no) (in_bom yes) (on_board yes) (dnp no)
-    (property "Reference" "LED1" (at 1041.4 495.3 0))
-    (property "Value" "Red LED" (at 1041.4 520.7 0))
-    (property "Footprint" "" (at 1016.0 508.0 0))
-    (property "Datasheet" "~" (at 1016.0 508.0 0))
+    (property "Reference" "LED1" (at 1025.4 487.3 0))
+    (property "Value" "Red" (at 1025.4 512.7 0))
+    (property "Footprint" "" (at 1000 500 0))
+    (property "Datasheet" "~" (at 1000 500 0))
     (pin "1")
     (pin "2")
   )
-  (symbol (lib_id "power:VCC") (at 254.0 254.0 0) (unit 1)
+  (symbol (lib_id "power:VCC") (at 250 250 0) (unit 1)
     (exclude_from_sim no) (in_bom yes) (on_board yes) (dnp no)
-    (property "Reference" "#PWR01" (at 254.0 228.6 0))
-    (property "Value" "VCC" (at 254.0 289.56 0))
-    (property "Footprint" "" (at 254.0 254.0 0))
-    (property "Datasheet" "" (at 254.0 254.0 0))
+    (property "Reference" "#PWR01" (at 250 224.6 0))
+    (property "Value" "VCC" (at 250 285.56 0))
+    (property "Footprint" "" (at 250 250 0))
+    (property "Datasheet" "" (at 250 250 0))
     (pin "1")
   )
-  (symbol (lib_id "power:GND") (at 254.0 1016.0 0) (unit 1)
+  (symbol (lib_id "power:GND") (at 250 750 0) (unit 1)
     (exclude_from_sim no) (in_bom yes) (on_board yes) (dnp no)
-    (property "Reference" "#PWR02" (at 254.0 990.6 0))
-    (property "Value" "GND" (at 254.0 1051.56 0))
-    (property "Footprint" "" (at 254.0 1016.0 0))
-    (property "Datasheet" "" (at 254.0 1016.0 0))
+    (property "Reference" "#PWR02" (at 250 724.6 0))
+    (property "Value" "GND" (at 250 785.56 0))
+    (property "Footprint" "" (at 250 750 0))
+    (property "Datasheet" "" (at 250 750 0))
     (pin "1")
   )
