File: tests/visual_output/test_circuit.kicad_sch (KiCad schematic)
At the start: 2 parts

Commit message: feat: implement comprehensive boundary validation system for component positioning
This commit implements a complete boundary validation system that addresses
the high priority task from TASKS.md: "Add automated boundary validation
for component positioning".

New Features:
- BoundaryValidator utility class with A4 schematic bounds checking
- ValidationTools for project-level validation of existing schematics
- Integration into circuit generation pipeline with auto-correction
- Comprehensive validation reporting (text and JSON formats)
- Pre-generation validation checks for all circuit creation tools

Core Components:
- kicad_mcp/utils/boundary_validator.py: Core validation logic with severity levels
- kicad_mcp/tools/validation_tools.py: Project validation tools
- kicad_mcp/utils/coordinate_converter.py: Enhanced coordinate utilities

Integration Points:
- circuit_tools.py: Integrated into add_component and create_wire_connection
- text_to_schematic.py: Pre-generation validation with auto-correction
- sexpr_generator.py: Enhanced position validation in layout manager

Validation Features:
- A4 page bounds compliance (297x210mm with 20mm margins)
- Component-aware validation with different rules per component type
- Auto-correction of out-of-bounds positions using layout manager
- Validation severity levels (ERROR/WARNING/INFO)
- Comprehensive reporting with suggested corrections

Testing:
- 45+ unit tests for BoundaryValidator
- Integration tests for end-to-end validation workflows
- Visual validation tests for schematic generation

This system prevents coordinate issues that were previously causing problems
with component positioning in KiCad schematics and ensures all generated
circuits comply with A4 schematic standards.

🤖 Generated with Claude Code

Co-Authored-By: Claude <noreply@anthropic.com>
Changed lines of the file:
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@@
 (kicad_sch
-  (version 20230121)
+  (version 20240618)
   (generator kicad-mcp)
   (paper "A4")
@@
     (company "")
   )
-  (symbol (lib_id "Device:R") (at 500 500 0) (unit 1)
+  (symbol (lib_id "Device:R") (at 50.0 50.0 0) (unit 1)
     (exclude_from_sim no) (in_bom yes) (on_board yes) (dnp no)
-    (property "Reference" "R1" (at 525.4 487.3 0))
-    (property "Value" "1kΩ" (at 525.4 512.7 0))
-    (property "Footprint" "" (at 500 500 0))
-    (property "Datasheet" "~" (at 500 500 0))
+    (property "Reference" "R1" (at 75.4 37.3 0))
+    (property "Value" "1kΩ" (at 75.4 62.7 0))
+    (property "Footprint" "" (at 50.0 50.0 0))
+    (property "Datasheet" "~" (at 50.0 50.0 0))
     (pin "1")
     (pin "2")
   )
-  (symbol (lib_id "Device:LED") (at 1000 500 0) (unit 1)
+  (symbol (lib_id "Device:LED") (at 100.0 50.0 0) (unit 1)
     (exclude_from_sim no) (in_bom yes) (on_board yes) (dnp no)
-    (property "Reference" "LED1" (at 1025.4 487.3 0))
-    (property "Value" "Red" (at 1025.4 512.7 0))
-    (property "Footprint" "" (at 1000 500 0))
-    (property "Datasheet" "~" (at 1000 500 0))
+    (property "Reference" "LED1" (at 125.4 37.3 0))
+    (property "Value" "Red" (at 125.4 62.7 0))
+    (property "Footprint" "" (at 100.0 50.0 0))
+    (property "Datasheet" "~" (at 100.0 50.0 0))
     (pin "1")
     (pin "2")
   )
-  (symbol (lib_id "power:VCC") (at 250 250 0) (unit 1)
+  (symbol (lib_id "power:VCC") (at 25.0 25.0 0) (unit 1)
     (exclude_from_sim no) (in_bom yes) (on_board yes) (dnp no)
-    (property "Reference" "#PWR01" (at 250 224.6 0))
-    (property "Value" "VCC" (at 250 285.56 0))
-    (property "Footprint" "" (at 250 250 0))
-    (property "Datasheet" "" (at 250 250 0))
+    (property "Reference" "#PWR01" (at 25.0 -0.3999999999999986 0))
+    (property "Value" "VCC" (at 25.0 60.56 0))
+    (property "Footprint" "" (at 25.0 25.0 0))
+    (property "Datasheet" "" (at 25.0 25.0 0))
     (pin "1")
   )
-  (symbol (lib_id "power:GND") (at 250 750 0) (unit 1)
+  (symbol (lib_id "power:GND") (at 25.0 75.0 0) (unit 1)
     (exclude_from_sim no) (in_bom yes) (on_board yes) (dnp no)
-    (property "Reference" "#PWR02" (at 250 724.6 0))
-    (property "Value" "GND" (at 250 785.56 0))
-    (property "Footprint" "" (at 250 750 0))
-    (property "Datasheet" "" (at 250 750 0))
+    (property "Reference" "#PWR02" (at 25.0 49.6 0))
+    (property "Value" "GND" (at 25.0 110.56 0))
+    (property "Footprint" "" (at 25.0 75.0 0))
+    (property "Datasheet" "" (at 25.0 75.0 0))
     (pin "1")
   )
